Commit message: description: fix broken URIs

File: tams_pr2_description/urdf/base_v0/base.urdf.xacro (robot description, xacro)
@@ -5,7 +5,7 @@
        xmlns:xacro="http://ros.org/wiki/xacro">
   <include filename="$(find pr2_description)/urdf/sensors/hokuyo_lx30_laser.urdf.xacro" />
-  <include filename="$(find race_pr2_description)/urdf/sensors/tray_hokuyo_lx30_laser.urdf.xacro" />
   <include filename="$(find pr2_description)/urdf/base_v0/base.gazebo.xacro" />
   <include filename="$(find pr2_description)/urdf/base_v0/base.transmission.xacro" />
+  <include filename="$(find tams_pr2_description)/urdf/sensors/tray_hokuyo_lx30_laser.urdf.xacro" />
   <!-- DATA SOURCES -->
   <!-- all link offsets, CG, limits are obtained from Function Engineering spreadsheet 090224_link_data.xls unless stated otherwise -->
@@ -167,5 +167,5 @@
         <origin xyz="-0.08 0 -0.295" rpy="0 0 0.0" />
         <geometry>
-          <mesh filename="package://race_pr2_description/meshes/base_v0/tray.dae" />
+          <mesh filename="package://tams_pr2_description/meshes/base_v0/tray.dae" />
         </geometry>
         <material name="White" />
@@ -175,5 +175,5 @@
         <origin xyz="-0.08 0 -0.295" rpy="0 0 0.0" />
        <geometry>
-          <mesh filename="package://race_pr2_description/meshes/base_v0/tray.dae" />
+          <mesh filename="package://tams_pr2_description/meshes/base_v0/tray.dae" />
           <!--Dummy box as otherwise tray is not rendered in Gazebo-->
           <!--<box size="0.0001 0.0001 0.0001" />-->

Commit message: improve tray description&model

File: tams_pr2_description/urdf/base_v0/base.urdf.xacro (robot description, xacro)
@@ -167,7 +167,9 @@
         <origin xyz="-0.08 0 -0.295" rpy="0 0 0.0" />
         <geometry>
-          <mesh filename="package://tams_pr2_description/meshes/base_v0/tray.dae" />
-        </geometry>
-        <material name="White" />
+          <mesh filename="package://tams_pr2_description/meshes/base_v0/tray.stl" />
+        </geometry>
+        <material name="Metallic">
+          <texture filename="package://tams_pr2_description/meshes/base_v0/metallic.png" />
+        </material>
       </visual>
       <!--Collision is defined in base_L.stl and part of the base collision model-->
@@ -175,7 +177,5 @@
         <origin xyz="-0.08 0 -0.295" rpy="0 0 0.0" />
        <geometry>
-          <mesh filename="package://tams_pr2_description/meshes/base_v0/tray.dae" />
-          <!--Dummy box as otherwise tray is not rendered in Gazebo-->
-          <!--<box size="0.0001 0.0001 0.0001" />-->
+          <mesh filename="package://tams_pr2_description/meshes/base_v0/tray_L.stl" />
        </geometry>
       </collision>

Commit message: provide a neat visual tray

File: tams_pr2_description/urdf/base_v0/base.urdf.xacro (robot description, xacro)
@@ -165,5 +165,5 @@
       </inertial>
       <visual>
-        <origin xyz="-0.08 0 -0.295" rpy="0 0 0.0" />
+        <origin xyz="0.0 0 0.0" rpy="0 0 0.0" />
         <geometry>
           <mesh filename="package://tams_pr2_description/meshes/base_v0/tray.stl" />
@@ -173,10 +173,9 @@
         </material>
       </visual>
-      <!--Collision is defined in base_L.stl and part of the base collision model-->
-      <collision>
-        <origin xyz="-0.08 0 -0.295" rpy="0 0 0.0" />
-       <geometry>
+      <collision>
+        <origin xyz="-0.08 0 -0.290" rpy="0 0 0.0" />
+        <geometry>
           <mesh filename="package://tams_pr2_description/meshes/base_v0/tray_L.stl" />
-       </geometry>
+        </geometry>
       </collision>
     </link>
