Commit message: Make transmissions ros_control compatible
The transmission style changed for ros_control, the transmissions
need a type element a joint element with a hardware interface and
an actuator.

File: tams_pr2_description/urdf/ft_forearm/ft_forearm.transmission.xacro (robot description, xacro)
@@ -6,5 +6,12 @@
   <xacro:macro name="pr2_ft_forearm_transmission" params="side">
     <!-- Wrist flex , Wrist roll -->
-    <transmission type="pr2_mechanism_model/WristTransmission" name="${side}_wrist_trans">
+    <transmission name="${side}_wrist_trans">
+      <type>pr2_mechanism_model/WristTransmission</type>
+      <joint name="${side}_wrist_flex_joint">
+        <hardwareInterface>EffortJointInterface</hardwareInterface>
+      </joint>
+      <actuator name="${side}_wrist_r_motor">
+        <mechanicalReduction>1.0</mechanicalReduction>
+      </actuator>
       <rightActuator name="${side}_wrist_r_motor" mechanicalReduction="${624/35*54/16}"/>
       <leftActuator name="${side}_wrist_l_motor"  mechanicalReduction="${624/35*54/16}"/>
