Commit message: rectify ridiculous collision geometry for xtion

File: tams_pr2_description/urdf/xtion_camera.urdf.xacro (robot description, xacro)
@@ -27,7 +27,7 @@
       </visual>
       <collision>
-        <origin xyz="0.0 0.0 0" rpy="0 0 0"/>
+        <origin xyz="-0.02 -0.023 0.01" rpy="0 0 0"/>
         <geometry>
-          <sphere radius="0.1"/>
+          <box size="0.04 0.19 0.03" />
         </geometry>
       </collision>
