Commit message: Add Pixel 6 Pro holder; adjust Pixel 6 Pro position.

File: tams_pr2_description/urdf/tams_head_additions.urdf.xacro (robot description, xacro)
@@ -89,9 +89,30 @@
   </joint>
   <!-- Google Pixel 6 Pro phone - not updated yet for current holder placement-->
+  <!-- head top mounting plate is 95mm above head_plate_frame, center of phone is xxmm above the plate -->
   <xacro:pixel_6_pro name="pixel_6_pro" />
   <joint name="pixel_6_pro_mount_joint" type="fixed">
     <parent link="${parent}" />
     <child link="pixel_6_pro" />
-    <origin xyz="0.050 0.0 0.050" rpy="0. 0. 0." />
+    <origin xyz="0.052 0.0 ${0.095+0.0105}" rpy="0. 0. 0." />
+  </joint>
+  <link name="pixel_6_pro_holder" >
+     <!-- mesh for visual, no collision model (covered by generic collider) -->
+    <visual>
+      <origin xyz="0.0 0.0 0.0" rpy="0 0 1.571" />
+      <material name="pixel_6_pro_holder_material_white">
+        <color rgba="0.95 0.95 0.95 1.0" />
+      </material>
+      <geometry>
+        <mesh filename="package://tams_pr2_description/meshes/pr2_pixel_6_pro_holder_v3.stl" scale="0.001 0.001 0.001" />
+      </geometry>
+    </visual>
+    <!--
+    <collision/>
+    -->
+  </link>
+  <joint name="pixel_6_pro_holder_joint" type="fixed">
+    <parent link="${parent}" />
+    <child link="pixel_6_pro_holder" />
+    <origin xyz="${-2.5*0.0254} 0.0 ${0.0505}" rpy="0. 0. 0." />
   </joint>
 </xacro:macro>

Commit message: update calibration + add azure calibration offsets

File: tams_pr2_description/urdf/tams_head_additions.urdf.xacro (robot description, xacro)
@@ -61,5 +61,5 @@
     <parent link="${parent}" />
     <child link="${azure_kinect_name}_camera_base" />
-    <origin xyz="${0.0+0.022+0.026} 0.0 ${0.095 + 0.068 + 0.008}" rpy="0 0 0" />
+    <origin xyz="${0.0+0.022+0.026+calib['azure_kinect_camera_base_pos_x']} ${0.0+calib['azure_kinect_camera_base_pos_y']} ${0.095 + 0.068 + 0.008 + calib['azure_kinect_camera_base_pos_z']}" rpy="${calib['azure_kinect_camera_base_rot_r']} ${calib['azure_kinect_camera_base_rot_p']} ${calib['azure_kinect_camera_base_rot_y']}" />
   </joint>
   <link name="${azure_kinect_name}_holder" >
