Commit message: systematically disable casters
... instead of selectively disabling fl.
The main reason for this change is that bl also generated power failure status reports
recently. After fixing the slip rings this is what is needed to revert to a mobile base:

- reenabling caster calibration on startup (in calibrate_pr2.py)
- changing the fixed_wheels property to false (in tams_base.urdf.xacro)
- and re-enabling the base_controller base_odometry controllers (in pr2_default_controllers.launch)
- re-enabling the analyzers for the joints in the diagnostics board (analyzers.yaml)

File: tams_pr2_description/urdf/tams_base.urdf.xacro (robot description, xacro)
@@ -8,4 +8,5 @@
   <!-- all link geometry sizes are obtained from Function provided CAD model unless stated otherwise -->
   <!-- all simplified collision geometry are hand approximated from CAD model, sometimes from respective bounding boxes -->
+  <xacro:property name="fixed_wheels" value="true" />
   <xacro:property name="M_PI" value="3.1415926535897931" />
   <xacro:property name="caster_offset_x" value="0.2246" />
@@ -36,5 +37,5 @@
   <!--                                                      -->
   <xacro:macro name="pr2_wheel_v0" params="suffix parent reflect">
-    <xacro:if value="${parent == 'fl_caster'}">
+    <xacro:if value="${fixed_wheels}">
     <joint name="${parent}_${suffix}_wheel_joint" type="fixed">
       <origin xyz="0 ${reflect*caster_wheel_offset_y} 0" rpy="0 0 0" />
@@ -43,5 +44,5 @@
     </joint>
     </xacro:if>
-    <xacro:unless value="${parent == 'fl_caster'}">
+    <xacro:unless value="${fixed_wheels}">
     <joint name="${parent}_${suffix}_wheel_joint" type="continuous">
       <axis xyz="0 1 0" />
@@ -53,4 +54,5 @@
       <child link="${parent}_${suffix}_wheel_link"/>
     </joint>
+    <xacro:pr2_wheel_transmission_v0 parent="${parent}" suffix="${suffix}" reflect="${reflect}" />
     </xacro:unless>
     <link name="${parent}_${suffix}_wheel_link">
@@ -77,11 +79,8 @@
     <!-- extensions -->
     <xacro:pr2_wheel_gazebo_v0 parent="${parent}" suffix="${suffix}" />
-    <xacro:unless value="${parent == 'fl_caster'}">
-    <xacro:pr2_wheel_transmission_v0 parent="${parent}" suffix="${suffix}" reflect="${reflect}" />
-    </xacro:unless>
   </xacro:macro>
   <!-- Macro for PR2 Caster hub only -->
   <xacro:macro name="pr2_caster_hub_v0" params="suffix parent *origin ref_position" >
-    <xacro:if value="${suffix == 'fl_caster'}">
+    <xacro:if value="${fixed_wheels}">
     <joint name="${suffix}_rotation_joint" type="fixed">
       <xacro:insert_block name="origin" />
@@ -90,5 +89,5 @@
     </joint>
     </xacro:if>
-    <xacro:unless value="${suffix == 'fl_caster'}">
+    <xacro:unless value="${fixed_wheels}">
     <joint name="${suffix}_rotation_joint" type="continuous">
       <axis xyz="0 0 1" />
@@ -101,4 +100,5 @@
       <child link="${suffix}_rotation_link" />
     </joint>
+    <xacro:pr2_caster_transmission_v0 suffix="${suffix}" />
     </xacro:unless>
     <link name="${suffix}_rotation_link">
@@ -124,7 +124,4 @@
     </link>
     <!-- extensions -->
-    <xacro:unless value="${suffix == 'fl_caster'}">
-    <xacro:pr2_caster_transmission_v0 suffix="${suffix}" />
-    </xacro:unless>
   </xacro:macro>
   <xacro:macro name="pr2_caster_v0" params="suffix parent *origin ref_position">
