Commit message: make collision geometry consistent
everything that is visible from the outside *should* be checked for collisions.

Everything else should not be visible either.

File: tams_pr2_description/robots/calibrated.urdf (robot description, URDF)
Before this commit: robot tams_pr2, 127 links, 126 joints
Links:
- link double_stereo_link: geometry 
- link l_force_torque_link: geometry collision cylinder length=0.0356 radius=0.0225; visual cylinder length=0.0356 radius=0.0225
- link sensor_mount_link: geometry 

File: tams_pr2_description/urdf/ft_forearm/ft_ati_mini45.urdf.xacro (robot description, xacro)
@@ -21,4 +21,11 @@
         <material name="Grey"/>
       </visual>
+      <collision>
+        <origin rpy="0 0 0" xyz="0 0 -0.0120"/>
+        <geometry>
+         <cylinder length="0.0356" radius="0.0225"/>
+        </geometry>
+        <material name="Grey"/>
+      </collision>
     </link>
   </xacro:macro>

Commit message: update calibrated urdf w.r.t. xtion changes

File: tams_pr2_description/robots/calibrated.urdf (robot description, URDF)
Before this commit: robot tams_pr2, 127 links, 126 joints
Links:
- removed link head_mount_kinect_ir_link
- removed link head_mount_kinect_ir_optical_frame
- removed link head_mount_kinect_rgb_link
- removed link head_mount_kinect_rgb_optical_frame
- link head_mount_link: geometry collision box size=0.04 0.19 0.03; visual mesh filename=package://tams_pr2_description/meshes/xtion/xtion.stl
Joints:
- removed joint head_mount_kinect_ir_joint
- removed joint head_mount_kinect_ir_optical_frame_joint
- removed joint head_mount_kinect_rgb_joint
- removed joint head_mount_kinect_rgb_optical_frame_joint

Commit message: provide reasonable collision checking for kinect2 spoiler

File: tams_pr2_description/robots/calibrated.urdf (robot description, URDF)
Before this commit: robot tams_pr2, 123 links, 122 joints
Links:
- link head_mount_kinect2_link: geometry collision box size=0.12 0.3 0.2; visual mesh filename=package://pr2_description/meshes/sensors/kinect2_v0/kinect2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 scale=0.001 0.001 0.001

Commit message: new generated calibrated urdf by rixi.urdf.xacro
here are main changes:
1.hardwareInterface
  <!-- extensions -->
  <transmission name="fl_caster_rotation_trans">
    <type>pr2_mechanism_model/SimpleTransmission</type>
    <actuator name="fl_caster_rotation_motor">
      <mechanicalReduction>-79.2380952381</mechanicalReduction>
    </actuator>
    <joint name="fl_caster_rotation_joint">
      <hardwareInterface>hardware_interface/EffortJointInterface</hardwareInterface>
    </joint>
  </transmission>
---------------------------------------------------------------
  <transmission name="fl_caster_rotation_trans">
    <type>pr2_mechanism_model/SimpleTransmission</type>
    <actuator name="fl_caster_rotation_motor">
      <mechanicalReduction>-79.2380952381</mechanicalReduction>
    </actuator>
    <joint name="fl_caster_rotation_joint">
      <hardwareInterface>EffortJointInterface</hardwareInterface>
    </joint>
  </transmission>

2. name changes of head_mount_xtion_joint and head_mount_xtion_link
  <joint name="head_mount_xtion_joint" type="fixed">
    <origin rpy="0 0 0" xyz="0.03 0.02 0.091746"/>
    <parent link="head_plate_frame"/>
    <child link="head_mount_xtion_link"/>
  </joint>
---------------------------------------------------------------
  <joint name="head_mount_joint" type="fixed">
    <origin rpy="0 0 0" xyz="0.03 0.02 0.091746" />
    <parent link="head_plate_frame" />
    <child link="head_mount_link" />
  </joint>

3. folder change of sr_description meshes
      <geometry name="rh_forearm_visual">
        <mesh filename="package://sr_description/meshes/hand/forearm.dae" scale="0.001 0.001 0.001"/>
      </geometry>
---------------------------------------------------------------
    <geometry name="rh_forearm_visual">
        <mesh filename="package://sr_description/hand/model/forearm.dae" scale="0.001 0.001 0.001" />
      </geometry>

4. a new rh_ee_fixed_joint joint
  <joint name="rh_ee_fixed_joint" type="fixed">
    <parent link="rh_palm"/>
    <child link="rh_manipulator"/>
    <origin rpy="0.0 0.0 0.0" xyz="0.0 0.0 0.05"/>
  </joint>
  <link name="rh_manipulator"/>

5. a new joint and a new link about the palm imu
  <link name="rh_imu"/>
  <joint name="rh_palm_to_imu" type="fixed">
    <parent link="rh_palm"/>
    <child link="rh_imu"/>
    <origin rpy="-1.5707963 3.141592 0.0" xyz="0.01785 0.00765 0.049125"/>
  </joint>
  <sensor name="rh_imu" update_rate="100">
    <parent link="rh_imu"/>
    <origin rpy="0 0 0" xyz="0 0 0"/>
    <imu/>
  </sensor>

6. joint range changes of Shadow hand joint3
  <joint name="rh_MFJ3" type="revolute">
    <parent link="rh_mfknuckle"/>
    <child link="rh_mfproximal"/>
    <origin rpy="0 0 0" xyz="0 0 0"/>
    <axis xyz="1 0 0"/>
    <limit effort="2" lower="-0.261799387799" upper="1.57079632679" velocity="2.0"/>
    <dynamics damping="0.1"/>
  </joint>

7. from 'true' to 'True' for turnGravityOff
  <gazebo reference="rh_wrist">
    <turnGravityOff>True</turnGravityOff>
  </gazebo>
---------------------------------------------------------------
<gazebo reference="rh_wrist">
    <turnGravityOff>true</turnGravityOff>
  </gazebo>

8. delete lots of useless white space
9. some description are changed or updated

File: tams_pr2_description/robots/calibrated.urdf (robot description, URDF)
Before this commit: robot tams_pr2, 123 links, 122 joints
Links:
- removed link head_mount_link
- added link head_mount_xtion_link, mass 0.1; collision box size=0.04 0.19 0.03; visual mesh filename=package://tams_pr2_description/meshes/xtion/xtion.stl
- added link rh_imu
- added link rh_manipulator
- link rh_ffdistal: geometry collision mesh filename=package://sr_description/meshes/hand/biotacs/biotac_decimat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 scale=0.0254 0.0254 0.0254; visual mesh filename=package://sr_description/meshes/hand/biotacs/biotac_decimat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 scale=0.0254 0.0254 0.0254
- link rh_ffknuckle: geometry collision cylinder length=0.014 radius=0.007; visual mesh filename=package://sr_description/meshes/hand/knuckle.dae scale=0.001 0.001 0.001
- link rh_ffmiddle: geometry collision box size=0.001 0.001 0.001; visual mesh filename=package://sr_description/meshes/hand/biotacs/biotac_finger_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 scale=1 1 1
- link rh_ffproximal: geometry collision cylinder length=0.040 radius=0.007; visual mesh filename=package://sr_description/meshes/hand/F3.dae scale=0.001 0.001 0.001
- link rh_forearm: geometry collision box size=0.07 0.07 0.07; collision cylinder length=0.184 radius=0.07
- link rh_lfdistal: geometry collision mesh filename=package://sr_description/meshes/hand/biotacs/biotac_decimat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 scale=0.0254 0.0254 0.0254; visual mesh filename=package://sr_description/meshes/hand/biotacs/biotac_decimat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 scale=0.0254 0.0254 0.0254
- link rh_lfknuckle: geometry collision cylinder length=0.014 radius=0.007; visual mesh filename=package://sr_description/meshes/hand/knuckle.dae scale=0.001 0.001 0.001
- link rh_lfmetacarpal: geometry collision box size=0.018 0.024 0.040; visual mesh filename=package://sr_description/meshes/hand/lfmetacarpal.dae scale=0.001 0.001 0.001
- link rh_lfmiddle: geometry collision box size=0.001 0.001 0.001; visual mesh filename=package://sr_description/meshes/hand/biotacs/biotac_finger_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 scale=1 1 1
- link rh_lfproximal: geometry collision cylinder length=0.040 radius=0.007; visual mesh filename=package://sr_description/meshes/hand/F3.dae scale=0.001 0.001 0.001
- link rh_mfdistal: geometry collision mesh filename=package://sr_description/meshes/hand/biotacs/biotac_decimat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 scale=0.0254 0.0254 0.0254; visual mesh filename=package://sr_description/meshes/hand/biotacs/biotac_decimat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 scale=0.0254 0.0254 0.0254
- link rh_mfknuckle: geometry collision cylinder length=0.014 radius=0.007; visual mesh filename=package://sr_description/meshes/hand/knuckle.dae scale=0.001 0.001 0.001
- link rh_mfmiddle: geometry collision box size=0.001 0.001 0.001; visual mesh filename=package://sr_description/meshes/hand/biotacs/biotac_finger_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 scale=1 1 1
- link rh_mfproximal: geometry collision cylinder length=0.040 radius=0.007; visual mesh filename=package://sr_description/meshes/hand/F3.dae scale=0.001 0.001 0.001
- link rh_palm: geometry collision box size=0.018 0.024 0.004; collision box size=0.020 0.024 0.040
- link rh_rfdistal: geometry collision mesh filename=package://sr_description/meshes/hand/biotacs/biotac_decimat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 scale=0.0254 0.0254 0.0254; visual mesh filename=package://sr_description/meshes/hand/biotacs/biotac_decimat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 scale=0.0254 0.0254 0.0254
- link rh_rfknuckle: geometry collision cylinder length=0.014 radius=0.007; visual mesh filename=package://sr_description/meshes/hand/knuckle.dae scale=0.001 0.001 0.001
- link rh_rfmiddle: geometry collision box size=0.001 0.001 0.001; visual mesh filename=package://sr_description/meshes/hand/biotacs/biotac_finger_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 scale=1 1 1
- link rh_rfproximal: geometry collision cylinder length=0.040 radius=0.007; visual mesh filename=package://sr_description/meshes/hand/F3.dae scale=0.001 0.001 0.001
- link rh_thdistal: geometry collision mesh filename=package://sr_description/meshes/hand/biotacs/biotac_decimat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 scale=0.0254 0.0254 0.0254; visual mesh filename=package://sr_description/meshes/hand/biotacs/biotac_decimat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 scale=0.0254 0.0254 0.0254
- link rh_thmiddle: geometry collision box size=0.001 0.001 0.001; visual mesh filename=package://sr_description/meshes/hand/biotacs/biotac_thumb_a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 scale=0.001 0.001 0.001
- link rh_thproximal: geometry collision cylinder length=0.018 radius=0.012; visual mesh filename=package://sr_description/meshes/hand/TH3_z.dae scale=0.001 0.001 0.001
- link rh_wrist: geometry collision box size=0.027 0.018 0.010; collision box size=0.027 0.018 0.010
Joints:
- removed joint head_mount_joint
- added joint head_mount_xtion_joint: type fixed, parent head_plate_frame, child head_mount_xtion_link, origin xyz=0.03 0.02 0.091746 rpy=0 0 0
- added joint rh_ee_fixed_joint: type fixed, parent rh_palm, child rh_manipulator, origin xyz=0.0 0.0 0.05 rpy=0.0 0.0 0.0
- added joint rh_palm_to_imu: type fixed, parent rh_palm, child rh_imu, origin xyz=0.01785 0.00765 0.049125 rpy=-1.5707963 3.141592 0.0
- joint rh_FFJ3: limit lower=0 upper=1.57079632679 effort=2 velocity=2.0 -> lower=-0.261799387799 upper=1.57079632679 effort=2 velocity=2.0
- joint rh_LFJ3: limit lower=0 upper=1.57079632679 effort=2 velocity=2.0 -> lower=-0.261799387799 upper=1.57079632679 effort=2 velocity=2.0
- joint rh_MFJ3: limit lower=0 upper=1.57079632679 effort=2 velocity=2.0 -> lower=-0.261799387799 upper=1.57079632679 effort=2 velocity=2.0
- joint rh_RFJ3: limit lower=0 upper=1.57079632679 effort=2 velocity=2.0 -> lower=-0.261799387799 upper=1.57079632679 effort=2 velocity=2.0
