Commit message: feed customized calibration values into trixi.urdf.xacros

File: tams_pr2_description/robots/calibrated_202009_07.urdf (robot description, URDF)
Before this commit: robot tams_pr2, 125 links, 124 joints
Links:
- link base_footprint: mass None -> 1.0
- link head_mount_kinect2_ir_link: geometry collision sphere radius=0.0005; visual sphere radius=0.0005
- link head_mount_kinect2_rgb_link: geometry collision sphere radius=0.0005; visual sphere radius=0.0005

File: tams_pr2_description/robots/trixi.urdf.xacro (robot description, xacro)
@@ -33,9 +33,12 @@
   <xacro:include filename="$(find tams_pr2_description)/urdf/tams_pr2_shadow_adapter.urdf.xacro" />
   <xacro:include filename="$(find tams_pr2_description)/urdf/xtion_camera.urdf.xacro" />
-  <xacro:include filename="$(find sr_description)/hand/xacro/full_hand.urdf.xacro" />
-  <xacro:include filename="$(find sr_description)/other/xacro/gazebo/gazebo.urdf.xacro"/>
   <xacro:include filename="$(find pr2_description)/urdf/sensors/kinect2.urdf.xacro" />
   <xacro:include filename="$(find tams_pr2_description)/urdf/turn_gravity_off.urdf.xacro" />
   <xacro:include filename="$(find tams_motorhand_description)/urdf/tams_motorhand.urdf.xacro" />
+  <xacro:arg name="calib_config" default="$(find tams_pr2_description)/config/calibration_config.yaml" />
+  <xacro:property name="calib" value="${load_yaml('$(arg calib_config)')}"/>
+  <!-- TAMS' Shadow additions -->
+  <xacro:include filename="$(find sr_description)/hand/xacro/full_hand.urdf.xacro" />
+  <xacro:include filename="$(find sr_description)/other/xacro/gazebo/gazebo.urdf.xacro"/>
   <!-- Now we can start using the macros included above to define the actual PR2 -->
   <xacro:pr2_base_v0 name="base"/>
@@ -43,8 +46,10 @@
     <origin xyz="0.08 0 0.295" rpy="0 0 0" />
   </xacro:tams_pr2_tray>
-  <xacro:pr2_torso_v0 name="torso_lift" parent="base_link">
+  <xacro:pr2_torso_v0 name="torso_lift" parent="base_link" torso_calib_ref="${calib['torso_calib_ref']}">
     <origin xyz="-0.05 0 0.739675" rpy="0 0 0" />
   </xacro:pr2_torso_v0>
-  <xacro:pr2_head_v0 name="head" parent="torso_lift_link">
+  <xacro:pr2_head_v0 name="head" parent="torso_lift_link"
+                     head_pan_calib_ref="${calib['head_pan_calib_ref']}"
+                     head_tilt_calib_ref="${calib['head_tilt_calib_ref']}">
     <origin xyz="-0.01707 0.0 0.38145"
             rpy="0.0 0.0 0.0" />
@@ -69,8 +74,13 @@
   </xacro:pr2_tilting_laser_v0>
   <!-- This is a common convention, to use a reflect parameter that equals +-1 to distinguish left from right -->
-  <xacro:pr2_shoulder_v0 side="r" reflect="-1" parent="torso_lift_link">
+  <xacro:pr2_shoulder_v0 side="r" reflect="-1" parent="torso_lift_link"
+                         shoulder_pan_calib_ref="${calib['r_shoulder_pan_calib_ref']}"
+                         shoulder_lift_calib_ref="${calib['r_shoulder_lift_calib_ref']}"
+                         upper_arm_roll_calib_ref="${calib['r_upper_arm_roll_calib_ref']}">
     <origin xyz="0.0 -0.188 0.0" rpy="0 0 0" />
   </xacro:pr2_shoulder_v0>
-  <xacro:pr2_upper_arm_v0 side="r" reflect="-1" parent="r_upper_arm_roll_link"/>
+  <xacro:pr2_upper_arm_v0 side="r" reflect="-1" parent="r_upper_arm_roll_link"
+                          forearm_roll_calib_ref="${calib['r_forearm_roll_calib_ref']}"
+                          elbow_flex_calib_ref="${calib['r_elbow_flex_calib_ref']}"  />
   <xacro:tams_pr2_shadow_adapter name="rh_adapter" parent="r_forearm_roll_link">
     <origin xyz="0.118 0 0" rpy="0 0 0" />
@@ -85,9 +95,16 @@
   <!-- This is necessary to simulate the 'floating' of the right arm-->
   <xacro:turn_rh_gravity_off enable="true"/>
-  <xacro:pr2_shoulder_v0 side="l" reflect="1" parent="torso_lift_link">
+  <xacro:pr2_shoulder_v0 side="l" reflect="1" parent="torso_lift_link"
+                         shoulder_pan_calib_ref="${calib['l_shoulder_pan_calib_ref']}"
+                         shoulder_lift_calib_ref="${calib['l_shoulder_lift_calib_ref']}"
+                         upper_arm_roll_calib_ref="${calib['l_upper_arm_roll_calib_ref']}">
     <origin xyz="0.0 0.188 0.0" rpy="0 0 0" />
   </xacro:pr2_shoulder_v0>
-  <xacro:pr2_upper_arm_v0 side="l" reflect="1" parent="l_upper_arm_roll_link"/>
-  <xacro:pr2_ft_forearm side="l" reflect="1" parent="l_forearm_roll_link">
+  <xacro:pr2_upper_arm_v0 side="l" reflect="1" parent="l_upper_arm_roll_link"
+                          forearm_roll_calib_ref="${calib['l_forearm_roll_calib_ref']}"
+                          elbow_flex_calib_ref="${calib['l_elbow_flex_calib_ref']}"  />
+  <xacro:pr2_ft_forearm side="l" reflect="1" parent="l_forearm_roll_link"
+                        wrist_flex_calib_ref="${calib['l_wrist_flex_calib_ref']}"
+                        wrist_roll_calib_ref="${calib['l_wrist_roll_calib_ref']}">
     <origin xyz="0 0 0" rpy="0 0 0" />
   </xacro:pr2_ft_forearm>

File: tams_pr2_description/urdf/ft_forearm/pr2_ft_forearm.urdf.xacro (robot description, xacro)
@@ -8,5 +8,7 @@
   <xacro:include filename="$(find tams_pr2_description)/urdf/ft_forearm/ft_ati_mini45.urdf.xacro" />
   <!-- ============================   Forearm   ============================ -->
-  <xacro:macro name="pr2_ft_forearm" params="side parent reflect *origin">
+  <xacro:macro name="pr2_ft_forearm" params="side parent reflect *origin
+    wrist_flex_calib_ref:=0
+    wrist_roll_calib_ref:=0">
     <joint name="${side}_forearm_joint" type="fixed">
       <xacro:insert_block name="origin" /> <!-- transform from parent link to this joint frame -->
@@ -42,5 +44,10 @@
       <safety_controller k_position="20" k_velocity="4" soft_upper_limit="${0.0 - 0.10}" soft_lower_limit="${-2.18 + 0.18}" />
       <dynamics damping="0.1" />
-      <calibration falling="${-0.5410521 + cal_r_wrist_flex_flag}" />
+      <xacro:unless value="${wrist_flex_calib_ref}">
+        <calibration  falling="${-0.5410521+cal_r_wrist_flex_flag}" />
+      </xacro:unless>
+      <xacro:if value="${wrist_flex_calib_ref}">
+        <calibration  falling="${wrist_flex_calib_ref}" />
+      </xacro:if>
       <origin xyz="0.321 0 0" rpy="0 0 0" />
       <parent link="${side}_forearm_link"/>
@@ -75,5 +82,10 @@
       <safety_controller k_velocity="2" />
       <dynamics damping="0.1" />
-      <calibration rising="${-M_PI / 2 + cal_r_wrist_roll_flag}" />
+      <xacro:unless value="${wrist_roll_calib_ref}">
+        <calibration rising="${-M_PI/2+cal_r_wrist_roll_flag}" />
+      </xacro:unless>
+      <xacro:if value="${wrist_roll_calib_ref}">
+        <calibration  rising="${wrist_roll_calib_ref}" />
+      </xacro:if>
       <origin xyz="0 0 0" rpy="0 0 0" />
       <parent link="${side}_wrist_flex_link"/>
