Commit message: rework description of tray
- use original pr2 base and add only the tray&tray laser scanner

File: tams_pr2_description/robots/trixi.urdf.xacro (robot description, xacro)
@@ -21,5 +21,5 @@
   <xacro:include filename="$(find pr2_description)/urdf/torso_v0/torso.urdf.xacro" />
   <!-- PR2 base -->
-  <xacro:include filename="$(find tams_pr2_description)/urdf/base_v0/base.urdf.xacro" />
+  <xacro:include filename="$(find pr2_description)/urdf/base_v0/base.urdf.xacro" />
   <!-- Head sensors -->
   <xacro:include filename="$(find pr2_description)/urdf/sensors/head_sensor_package.urdf.xacro" />
@@ -34,4 +34,6 @@
   <!-- materials for visualization -->
   <xacro:include filename="$(find pr2_description)/urdf/materials.urdf.xacro" />
+  <!-- TAMS' additions -->
+  <xacro:include filename="$(find tams_pr2_description)/urdf/tams_pr2_tray.urdf.xacro" />
   <!-- Now we can start using the macros included above to define the actual PR2 -->
   <!-- The first use of a macro.  This one was defined in base.urdf.xacro above.
@@ -43,4 +45,7 @@
        is the world frame). For more, see http://www.ros.org/wiki/xacro -->
   <xacro:pr2_base_v0 name="base"/>
+  <xacro:tams_pr2_tray name="tray" parent="base_link">
+    <origin xyz="0.08 0 0.295" rpy="0 0 0" />
+  </xacro:tams_pr2_tray>
   <xacro:pr2_torso_v0 name="torso_lift" parent="base_link">
     <origin xyz="-0.05 0 0.739675" rpy="0 0 0" />

File: tams_pr2_description/urdf/tams_hokuyo_lx30_laser.urdf.xacro (robot description, xacro)
@@ -1,13 +1,17 @@
 <?xml version="1.0"?>
+<!--
+pr2_description's hokuyo macro does not provide a visual link
+as the internal scanner is part of the pr2 base.
+-->
 <robot xmlns:sensor="http://playerstage.sourceforge.net/gazebo/xmlschema/#sensor"
        xmlns:controller="http://playerstage.sourceforge.net/gazebo/xmlschema/#controller"
        xmlns:interface="http://playerstage.sourceforge.net/gazebo/xmlschema/#interface"
        xmlns:xacro="http://ros.org/wiki/xacro">
-  <xacro:include filename="$(find tams_pr2_description)/urdf/sensors/tray_hokuyo_lx30_laser.gazebo.xacro" />
-  <xacro:macro name="tray_hokuyo_lx30_laser_v0" params="name parent *origin ros_topic update_rate min_angle max_angle">
+  <xacro:include filename="$(find pr2_description)/urdf/sensors/hokuyo_lx30_laser.gazebo.xacro" />
+  <xacro:macro name="tams_hokuyo_lx30_laser" params="name parent *origin ros_topic update_rate min_angle max_angle">
     <joint name="${name}_joint" type="fixed">
       <axis xyz="0 1 0" />
       <insert_block name="origin" />
-      <parent link="${parent}_link"/>
+      <parent link="${parent}"/>
       <child link="${name}_link"/>
     </joint>
@@ -21,6 +25,5 @@
       <origin xyz="-0.01 0 -0.015" rpy="0 0 0" />
       <geometry>
-        <mesh filename="package://tams_pr2_description/meshes/hokuyo/hokuyo.dae" />
-        <!--box size="0.05 0.05 0.1" /-->
+        <mesh filename="package://tams_pr2_description/meshes/hokuyo.dae" />
       </geometry>
     </visual>
@@ -33,5 +36,5 @@
     </link>
     <!-- gazebo extensions -->
-    <xacro:tray_hokuyo_lx30_laser_gazebo_v0 name="${name}" ros_topic="${ros_topic}" update_rate="${update_rate}" min_angle="${min_angle}" max_angle="${max_angle}" />
+    <xacro:hokuyo_lx30_laser_gazebo_v0 name="${name}" ros_topic="${ros_topic}" update_rate="${update_rate}" min_angle="${min_angle}" max_angle="${max_angle}" />
   </xacro:macro>
 </robot>

Commit message: add ft-sensor to trixi
The sensor is officially included by patching a generated urdf.
This is total nonsense and probably got added to ease usage
by "pure PR2 users". This commit takes the .patch files
and makes them proper urdf.xacro files instead.

File: tams_pr2_description/robots/trixi.urdf.xacro (robot description, xacro)
@@ -35,4 +35,5 @@
   <!-- TAMS' additions -->
   <xacro:include filename="$(find tams_pr2_description)/urdf/tams_pr2_tray.urdf.xacro" />
+  <xacro:include filename="$(find tams_pr2_description)/urdf/ft_forearm/pr2_ft_forearm.urdf.xacro" />
   <!-- Now we can start using the macros included above to define the actual PR2 -->
   <xacro:pr2_base_v0 name="base"/>
@@ -111,8 +112,8 @@
   </xacro:pr2_shoulder_v0>
   <xacro:pr2_upper_arm_v0 side="l" reflect="1" parent="l_upper_arm_roll_link"/>
-  <xacro:pr2_forearm_v0 side="l" reflect="1" parent="l_forearm_roll_link">
+  <xacro:pr2_ft_forearm side="l" reflect="1" parent="l_forearm_roll_link">
     <origin xyz="0 0 0" rpy="0 0 0" />
-  </xacro:pr2_forearm_v0>
-  <xacro:pr2_gripper_v0 reflect="1.0" side="l" parent="l_wrist_roll_link"
+  </xacro:pr2_ft_forearm>
+  <xacro:pr2_gripper_v0 reflect="1.0" side="l" parent="l_force_torque_link"
                screw_reduction="${4.0/1000.0}"
                gear_ratio="${(729.0/25.0)*(22.0/16.0)}"
@@ -125,5 +126,5 @@
                b="${43.3849/1000.0}"
                r="${91.5/1000.0}" >
-    <origin xyz="0 0 0" rpy="0 0 0" />
+    <origin xyz="0 0 0" rpy="0 1.5707963267948966 -1.2217304763960306" />
   </xacro:pr2_gripper_v0>
   <!-- Forearm cam Position is a guess, based on full robot calibration -->

Commit message: remove thermal camera from urdf

File: tams_pr2_description/robots/trixi.urdf.xacro (robot description, xacro)
@@ -76,12 +76,4 @@
     -->
   </xacro:kinect_prosilica_camera_swept_back_v0>
-  <!-- Base of Thermal Mount -->
-  <xacro:thermal_camera_v0 name="thermal_cam" image_format="R8G8B8"
-                           camera_name="thermal_cam" image_topic_name="image_raw"
-                           camera_info_topic_name="camera_info" parent="head_plate_frame" hfov="90"
-                           update_rate="5" focal_length="320" frame_id="thermal_cam_optical_frame"
-                           hack_baseline="0" image_width="640" image_height="480">
-    <origin xyz="-0.00 0.195 0.05" rpy="0 0 0" />
-  </xacro:thermal_camera_v0>
   <xacro:pr2_tilting_laser_v0 name="laser_tilt" parent="torso_lift_link" laser_calib_ref="0.0">
     <origin xyz="0.09893 0 0.227" rpy="0 0 0" />

Commit message: chop of right hand + add shadow adapter

File: tams_pr2_description/robots/trixi.urdf.xacro (robot description, xacro)
@@ -36,4 +36,5 @@
   <xacro:include filename="$(find tams_pr2_description)/urdf/tams_pr2_tray.urdf.xacro" />
   <xacro:include filename="$(find tams_pr2_description)/urdf/ft_forearm/pr2_ft_forearm.urdf.xacro" />
+  <xacro:include filename="$(find tams_pr2_description)/urdf/tams_pr2_shadow_adapter.urdf.xacro" />
   <!-- Now we can start using the macros included above to define the actual PR2 -->
   <xacro:pr2_base_v0 name="base"/>
@@ -84,20 +85,7 @@
   </xacro:pr2_shoulder_v0>
   <xacro:pr2_upper_arm_v0 side="r" reflect="-1" parent="r_upper_arm_roll_link"/>
-  <xacro:pr2_forearm_v0 side="r" reflect="-1" parent="r_forearm_roll_link">
-    <origin xyz="0 0 0" rpy="0 0 0" />
-  </xacro:pr2_forearm_v0>
-  <xacro:pr2_gripper_v0 reflect="-1.0" side="r" parent="r_wrist_roll_link"
-               screw_reduction="${4.0/1000.0}"
-               gear_ratio="${(729.0/25.0)*(22.0/16.0)}"
-               theta0="${3.6029*M_PI/180.0}"
-               phi0="${29.7089*M_PI/180.0}"
-               t0="${-0.1914/1000.0}"
-               L0="${37.5528/1000.0}"
-               h="${0.0/1000.0}"
-               a="${68.3698/1000.0}"
-               b="${43.3849/1000.0}"
-               r="${91.5/1000.0}" >
-    <origin xyz="0 0 0" rpy="0 0 0" />
-  </xacro:pr2_gripper_v0>
+  <xacro:tams_pr2_shadow_adapter name="r_hand_adapter" parent="r_forearm_roll_link">
+    <origin xyz="0.118 0 0" rpy="0 0 0" />
+  </xacro:tams_pr2_shadow_adapter>
   <xacro:pr2_shoulder_v0 side="l" reflect="1" parent="torso_lift_link">
     <origin xyz="0.0 0.188 0.0" rpy="0 0 0" />
@@ -129,10 +117,3 @@
     <origin xyz=".135 0 .044" rpy="${-M_PI/2} ${-32.25*M_PI/180} 0" />
   </xacro:wge100_camera_v0>
-  <xacro:wge100_camera_v0 name="r_forearm_cam" image_format="R8G8B8" camera_name="r_forearm_cam" image_topic_name="image_raw"
-                          camera_info_topic_name="camera_info"
-                          parent="r_forearm_roll_link" hfov="90" focal_length="320"
-                          frame_id="r_forearm_cam_optical_frame" hack_baseline="0"
-                          image_width="640" image_height="480">
-    <origin xyz=".135 0 .044" rpy="${M_PI/2} ${-32.25*M_PI/180} 0" />
-  </xacro:wge100_camera_v0>
 </robot>

Commit message: add shadow hand to trixi

File: tams_pr2_description/robots/trixi.urdf.xacro (robot description, xacro)
@@ -37,4 +37,5 @@
   <xacro:include filename="$(find tams_pr2_description)/urdf/ft_forearm/pr2_ft_forearm.urdf.xacro" />
   <xacro:include filename="$(find tams_pr2_description)/urdf/tams_pr2_shadow_adapter.urdf.xacro" />
+  <xacro:include filename="$(find sr_description)/hand/xacro/full_hand.urdf.xacro" />
   <!-- Now we can start using the macros included above to define the actual PR2 -->
   <xacro:pr2_base_v0 name="base"/>
@@ -88,4 +89,10 @@
     <origin xyz="0.118 0 0" rpy="0 0 0" />
   </xacro:tams_pr2_shadow_adapter>
+  <xacro:shadowhand muscletrans="false" muscle="false" bio="true" bt_sp="false" ubi="false" eli="false" reflect="1.0" prefix="r_hand_" lf="true" />
+  <joint name="r_hand_adapter_hand_joint" type="fixed">
+    <parent link="r_hand_adapter_link" />
+	 <child link="r_hand_forearm" />
+	 <origin xyz="0 0 0" rpy="0 ${-M_PI/2} ${M_PI}" />
+  </joint>
   <xacro:pr2_shoulder_v0 side="l" reflect="1" parent="torso_lift_link">
     <origin xyz="0.0 0.188 0.0" rpy="0 0 0" />

Commit message: trixi: add initial version of eyebrows

File: tams_pr2_description/robots/trixi.urdf.xacro (robot description, xacro)
@@ -24,5 +24,4 @@
   <!-- Head sensors -->
   <xacro:include filename="$(find pr2_description)/urdf/sensors/head_sensor_package.urdf.xacro" />
-  <xacro:include filename="$(find pr2_description)/urdf/sensors/kinect_prosilica_camera.urdf.xacro" />
   <!-- Camera sensors -->
   <xacro:include filename="$(find pr2_description)/urdf/sensors/wge100_camera.urdf.xacro" />
@@ -37,4 +36,5 @@
   <xacro:include filename="$(find tams_pr2_description)/urdf/ft_forearm/pr2_ft_forearm.urdf.xacro" />
   <xacro:include filename="$(find tams_pr2_description)/urdf/tams_pr2_shadow_adapter.urdf.xacro" />
+  <xacro:include filename="$(find tams_pr2_description)/urdf/xtion_camera.urdf.xacro" />
   <xacro:include filename="$(find sr_description)/hand/xacro/full_hand.urdf.xacro" />
   <!-- Now we can start using the macros included above to define the actual PR2 -->
@@ -57,4 +57,7 @@
     <origin xyz="0.0 0.0 0.0" rpy="0 0 0" />
   </xacro:pr2_head_sensor_package_v0>
+  <xacro:xtion_camera name="head_mount" parent="head_plate_frame">
+    <origin xyz="0.03 0.02 0.091746" rpy="0 0 0" />
+  </xacro:xtion_camera>
   <!-- Projector -->
   <xacro:projector_wg6802418_v0 name="projector_wg6802418" parent="head_plate_frame" >
@@ -62,20 +65,4 @@
     <origin xyz="0 0.110 0.0546" rpy="0 0 0" />
   </xacro:projector_wg6802418_v0>
-  <!-- Base of Kinect/Prosilica Mount -->
-  <xacro:kinect_prosilica_camera_swept_back_v0 name="head_mount" parent="head_plate_frame" >
-    <origin xyz="-0.137376 0 0.091746" rpy="0 0 0" />
-    <!--
-          Was -0.1 0 0.09225, -0.138 0 0.09225 looks good front back and sheet metal on bolt pattern,
-          -0.138 0 0.06225 is where Prosilica FOV just clears the head.
-          This is 30 mm (!) below the position in SolidWorks.
-          Lowering the Prosilica by this amount in SW makes the FOV hit around the aluminum / plastic junction.
-          Turns out that head_plate_frame is in some random position in space.
-          It is [0.0232 0 0.0645 from its parent, head_tilt_link.
-          The distance from head_plate_frame to the head_kinect_prosilica is 137.376 mm X and 91.746 mm Z.
-          So the origin should in fact be -0.137376 0 0.091746.
-          John is changing the Prosilica FOV based on my numbers.
-          Just need to roscd and svn up.
-    -->
-  </xacro:kinect_prosilica_camera_swept_back_v0>
   <xacro:pr2_tilting_laser_v0 name="laser_tilt" parent="torso_lift_link" laser_calib_ref="0.0">
     <origin xyz="0.09893 0 0.227" rpy="0 0 0" />

Commit message: add kinect2 to trixi urdf

File: tams_pr2_description/robots/trixi.urdf.xacro (robot description, xacro)
@@ -38,4 +38,5 @@
   <xacro:include filename="$(find tams_pr2_description)/urdf/xtion_camera.urdf.xacro" />
   <xacro:include filename="$(find sr_description)/hand/xacro/full_hand.urdf.xacro" />
+  <xacro:include filename="$(find pr2_description)/urdf/sensors/kinect2.urdf.xacro" />
   <!-- Now we can start using the macros included above to define the actual PR2 -->
   <xacro:pr2_base_v0 name="base"/>
@@ -111,3 +112,6 @@
     <origin xyz=".135 0 .044" rpy="${-M_PI/2} ${-32.25*M_PI/180} 0" />
   </xacro:wge100_camera_v0>
+  <xacro:kinect2_v0 name="head_mount" parent="head_plate_frame" >
+    <origin xyz="-0.137376 0 0.091746" rpy="0 0 0" />
+  </xacro:kinect2_v0>
 </robot>

Commit message: Change prefix of shadow related parts to match shadow convention

File: tams_pr2_description/robots/trixi.urdf.xacro (robot description, xacro)
@@ -74,11 +74,11 @@
   </xacro:pr2_shoulder_v0>
   <xacro:pr2_upper_arm_v0 side="r" reflect="-1" parent="r_upper_arm_roll_link"/>
-  <xacro:tams_pr2_shadow_adapter name="r_hand_adapter" parent="r_forearm_roll_link">
+  <xacro:tams_pr2_shadow_adapter name="rh_adapter" parent="r_forearm_roll_link">
     <origin xyz="0.118 0 0" rpy="0 0 0" />
   </xacro:tams_pr2_shadow_adapter>
-  <xacro:shadowhand muscletrans="false" muscle="false" bio="true" bt_sp="false" ubi="false" eli="false" reflect="1.0" prefix="r_hand_" lf="true" />
-  <joint name="r_hand_adapter_hand_joint" type="fixed">
-    <parent link="r_hand_adapter_link" />
-	 <child link="r_hand_forearm" />
+  <xacro:shadowhand muscletrans="false" muscle="false" bio="true" bt_sp="false" ubi="false" eli="false" reflect="1.0" prefix="rh_" lf="true" />
+  <joint name="rh_adapter_hand_joint" type="fixed">
+    <parent link="rh_adapter_link" />
+	 <child link="rh_forearm" />
 	 <origin xyz="0 0 0" rpy="0 ${-M_PI/2} ${M_PI}" />
   </joint>

Commit message: update xacro files to current standard

File: tams_pr2_description/robots/trixi.urdf.xacro (robot description, xacro)
@@ -1,8 +1,4 @@
 <?xml version="1.0"?>
-<robot xmlns:sensor="http://playerstage.sourceforge.net/gazebo/xmlschema/#sensor"
-       xmlns:controller="http://playerstage.sourceforge.net/gazebo/xmlschema/#controller"
-       xmlns:interface="http://playerstage.sourceforge.net/gazebo/xmlschema/#interface"
-       xmlns:xacro="http://playerstage.sourceforge.net/gazebo/xmlschema/#interface"
-       name="tams_pr2" >
+<robot xmlns:xacro="http://www.ros.org/wiki/xacro" name="tams_pr2" >
   <!-- The following included files set up definitions of parts of the robot body -->
   <!-- misc common stuff? -->

File: tams_pr2_description/urdf/ft_forearm/ft_ati_mini45.urdf.xacro (robot description, xacro)
@@ -1,12 +1,9 @@
 <?xml version="1.0"?>
-<robot xmlns:sensor="http://playerstage.sourceforge.net/gazebo/xmlschema/#sensor"
-       xmlns:controller="http://playerstage.sourceforge.net/gazebo/xmlschema/#controller"
-       xmlns:interface="http://playerstage.sourceforge.net/gazebo/xmlschema/#interface"
-       xmlns:xacro="http://ros.org/wiki/xacro">
+<robot xmlns:xacro="http://www.ros.org/wiki/xacro">
   <xacro:macro name="ft_at_mini45" params="side parent *origin">
     <joint name="${side}_force_torque_adapter_joint" type="fixed">
       <parent link="${parent}"/>
       <child link="${side}_force_torque_adapter_link"/>
-      <insert_block name="origin"/>
+      <xacro:insert_block name="origin"/>
     </joint>
     <link name="${side}_force_torque_adapter_link"/>

File: tams_pr2_description/urdf/ft_forearm/ft_forearm.transmission.xacro (robot description, xacro)
@@ -1,7 +1,4 @@
 <?xml version="1.0"?>
-<robot xmlns:sensor="http://playerstage.sourceforge.net/gazebo/xmlschema/#sensor"
-       xmlns:controller="http://playerstage.sourceforge.net/gazebo/xmlschema/#controller"
-       xmlns:interface="http://playerstage.sourceforge.net/gazebo/xmlschema/#interface"
-       xmlns:xacro="http://ros.org/wiki/xacro">
+<robot xmlns:xacro="http://www.ros.org/wiki/xacro">
   <xacro:macro name="pr2_ft_forearm_transmission" params="side">
     <!-- Wrist flex , Wrist roll -->

File: tams_pr2_description/urdf/ft_forearm/pr2_ft_forearm.urdf.xacro (robot description, xacro)
@@ -1,8 +1,4 @@
 <?xml version="1.0"?>
-<!-- XML namespaces -->
-<robot xmlns:sensor="http://playerstage.sourceforge.net/gazebo/xmlschema/#sensor"
-       xmlns:controller="http://playerstage.sourceforge.net/gazebo/xmlschema/#controller"
-       xmlns:interface="http://playerstage.sourceforge.net/gazebo/xmlschema/#interface"
-       xmlns:xacro="http://ros.org/wiki/xacro">
+<robot xmlns:xacro="http://www.ros.org/wiki/xacro">
   <!-- Things that are needed only for Gazebo (not the physical robot).  These include
        sensor and controller plugin specifications -->
@@ -14,5 +10,5 @@
   <xacro:macro name="pr2_ft_forearm" params="side parent reflect *origin">
     <joint name="${side}_forearm_joint" type="fixed">
-      <insert_block name="origin" /> <!-- transform from parent link to this joint frame -->
+      <xacro:insert_block name="origin" /> <!-- transform from parent link to this joint frame -->
       <parent link="${parent}"/>
       <child link="${side}_forearm_link"/>

File: tams_pr2_description/urdf/tams_hokuyo_lx30_laser.urdf.xacro (robot description, xacro)
@@ -4,13 +4,10 @@
 as the internal scanner is part of the pr2 base.
 -->
-<robot xmlns:sensor="http://playerstage.sourceforge.net/gazebo/xmlschema/#sensor"
-       xmlns:controller="http://playerstage.sourceforge.net/gazebo/xmlschema/#controller"
-       xmlns:interface="http://playerstage.sourceforge.net/gazebo/xmlschema/#interface"
-       xmlns:xacro="http://ros.org/wiki/xacro">
+<robot xmlns:xacro="http://www.ros.org/wiki/xacro">
   <xacro:include filename="$(find pr2_description)/urdf/sensors/hokuyo_lx30_laser.gazebo.xacro" />
   <xacro:macro name="tams_hokuyo_lx30_laser" params="name parent *origin ros_topic update_rate min_angle max_angle">
     <joint name="${name}_joint" type="fixed">
       <axis xyz="0 1 0" />
-      <insert_block name="origin" />
+      <xacro:insert_block name="origin" />
       <parent link="${parent}"/>
       <child link="${name}_link"/>

File: tams_pr2_description/urdf/tams_pr2_shadow_adapter.urdf.xacro (robot description, xacro)
@@ -1,7 +1,4 @@
 <?xml version="1.0"?>
-<robot xmlns:sensor="http://playerstage.sourceforge.net/gazebo/xmlschema/#sensor"
-       xmlns:controller="http://playerstage.sourceforge.net/gazebo/xmlschema/#controller"
-       xmlns:interface="http://playerstage.sourceforge.net/gazebo/xmlschema/#interface"
-       xmlns:xacro="http://ros.org/wiki/xacro">
+<robot xmlns:xacro="http://www.ros.org/wiki/xacro">
   <xacro:macro name="tams_pr2_shadow_adapter" params="name parent *origin">
     <link name="${name}_link">
@@ -28,5 +25,5 @@
     </link>
     <joint name="${name}_joint" type="fixed">
-      <insert_block name="origin" />
+      <xacro:insert_block name="origin" />
       <child link="${name}_link" />
       <parent link="${parent}"/>

File: tams_pr2_description/urdf/tams_pr2_tray.urdf.xacro (robot description, xacro)
@@ -1,7 +1,4 @@
 <?xml version="1.0"?>
-<robot xmlns:sensor="http://playerstage.sourceforge.net/gazebo/xmlschema/#sensor"
-       xmlns:controller="http://playerstage.sourceforge.net/gazebo/xmlschema/#controller"
-       xmlns:interface="http://playerstage.sourceforge.net/gazebo/xmlschema/#interface"
-       xmlns:xacro="http://ros.org/wiki/xacro">
+<robot xmlns:xacro="http://www.ros.org/wiki/xacro">
   <xacro:include filename="$(find tams_pr2_description)/urdf/tams_hokuyo_lx30_laser.urdf.xacro" />
   <xacro:macro name="tams_pr2_tray" params="name parent *origin">
@@ -31,5 +28,5 @@
     </link>
     <joint name="${name}_joint" type="fixed">
-      <insert_block name="origin" />
+      <xacro:insert_block name="origin" />
       <child link="${name}_link" />
       <parent link="${parent}"/>

File: tams_pr2_description/urdf/turn_gravity_off.urdf.xacro (robot description, xacro)
@@ -1,7 +1,4 @@
 <?xml version="1.0"?>
-<robot xmlns:sensor="http://playerstage.sourceforge.net/gazebo/xmlschema/#sensor"
-       xmlns:controller="http://playerstage.sourceforge.net/gazebo/xmlschema/#controller"
-       xmlns:interface="http://playerstage.sourceforge.net/gazebo/xmlschema/#interface"
-       xmlns:xacro="http://ros.org/wiki/xacro">
+<robot xmlns:xacro="http://www.ros.org/wiki/xacro">
   <xacro:macro name="turn_rh_gravity_off" params="enable">
     <gazebo reference="rh_wrist">

File: tams_pr2_description/urdf/xtion_camera.urdf.xacro (robot description, xacro)
@@ -1,12 +1,9 @@
 <?xml version="1.0"?>
-<root xmlns:sensor="http://playerstage.sourceforge.net/gazebo/xmlschema/#sensor"
-      xmlns:controller="http://playerstage.sourceforge.net/gazebo/xmlschema/#controller"
-      xmlns:interface="http://playerstage.sourceforge.net/gazebo/xmlschema/#interface"
-      xmlns:xacro="http://ros.org/wiki/xacro">
+<root xmlns:xacro="http://www.ros.org/wiki/xacro">
   <xacro:include filename="$(find pr2_description)/urdf/sensors/kinect_prosilica_camera.gazebo.xacro" />
-  <property name="ir_depth_rgb_offset_y" value="0.01"/> <!-- FIXME: what is this offset? -->
+  <xacro:property name="ir_depth_rgb_offset_y" value="0.01"/> <!-- FIXME: what is this offset? -->
   <xacro:macro name="xtion_camera" params="name parent *origin">
     <joint name="${name}_joint" type="fixed">
-      <insert_block name="origin" />
+      <xacro:insert_block name="origin" />
       <parent link="${parent}"/>
       <child link="${name}_link"/>
