Commit message: remove broken head frames from description
Apparently I copied the kinect1 description four years ago
and never adjusted the frames for the Xtion.

As we do not use it, just drop all the broken frames for now
and add a proper collision box around it instead.

File: tams_pr2_description/robots/trixi.urdf.xacro (robot description, xacro)
@@ -57,5 +57,5 @@
     <origin xyz="0.0 0.0 0.0" rpy="0 0 0" />
   </xacro:pr2_head_sensor_package_v0>
-  <xacro:xtion_camera name="head_mount" parent="head_plate_frame">
+  <xacro:xtion_camera name="head_mount_xtion" parent="head_plate_frame">
     <origin xyz="0.03 0.02 0.091746" rpy="0 0 0" />
   </xacro:xtion_camera>

File: tams_pr2_description/urdf/xtion_camera.urdf.xacro (robot description, xacro)
@@ -1,6 +1,5 @@
 <?xml version="1.0"?>
+<!-- TODO: if this should ever be used, the appropriate frames would need to be added first -->
 <root xmlns:xacro="http://www.ros.org/wiki/xacro">
-  <xacro:include filename="$(find pr2_description)/urdf/sensors/kinect_prosilica_camera.gazebo.xacro" />
-  <xacro:property name="ir_depth_rgb_offset_y" value="0.01"/> <!-- FIXME: what is this offset? -->
   <xacro:macro name="xtion_camera" params="name parent *origin">
     <joint name="${name}_joint" type="fixed">
@@ -33,56 +32,4 @@
       </collision>
     </link>
-    <joint name="${name}_kinect_ir_joint" type="fixed">
-      <origin xyz="-0.032267 0.0125 0.136453" rpy="0 0 0"/>
-      <parent link="${name}_link"/>
-      <child link="${name}_kinect_ir_link"/>
-    </joint>
-    <link name="${name}_kinect_ir_link" />
-    <joint name="${name}_kinect_ir_optical_frame_joint" type="fixed">
-      <origin xyz="${cal_kinect_x}            ${cal_kinect_y + ir_depth_rgb_offset_y}         ${cal_kinect_z}"
-                rpy="${-M_PI/2+cal_kinect_roll} ${0.0+cal_kinect_pitch} ${-M_PI/2+cal_kinect_yaw}" />
-      <parent link="${name}_kinect_ir_link"/>
-      <child link="${name}_kinect_ir_optical_frame"/>
-    </joint>
-    <link name="${name}_kinect_ir_optical_frame"/>
-    <!-- gazebo extensions -->
-    <xacro:kinect_ir_gazebo_v0 link_name="${name}_kinect_ir_link" frame_name="${name}_kinect_ir_optical_frame" camera_name="head_mount_kinect" />
-    <!-- kinect rgb sensor physical attachment -->
-    <joint name="${name}_kinect_rgb_joint" type="fixed">
-      <origin xyz="0 -0.03 0" rpy="0 0 0"/>
-      <parent link="${name}_kinect_ir_link"/>
-      <child link="${name}_kinect_rgb_link"/>
-    </joint>
-    <link name="${name}_kinect_rgb_link" >
-      <inertial>
-        <mass value="0.1" />
-        <origin xyz="0 0 0" rpy="0 0 0"/>
-        <inertia ixx="0.01"  ixy="0.0"  ixz="0.0"
-                 iyy="0.01"  iyz="0.0"
-                 izz="0.01" />
-      </inertial>
-      <visual>
-        <origin xyz="0.0 0.0 0" rpy="0 0 0"/>
-        <geometry>
-          <sphere radius="0.0005"/>
-        </geometry>
-      </visual>
-      <collision>
-        <origin xyz="0.0 0.0 0" rpy="0 0 0"/>
-        <geometry>
-          <sphere radius="0.0005"/>
-        </geometry>
-      </collision>
-    </link>
-    <!-- kinect rgb sensor frame -->
-    <joint name="${name}_kinect_rgb_optical_frame_joint" type="fixed">
-      <origin xyz="${cal_kinect_x}            ${cal_kinect_y}         ${cal_kinect_z}"
-                rpy="${-M_PI/2+cal_kinect_roll} ${0.0+cal_kinect_pitch} ${-M_PI/2+cal_kinect_yaw}" />
-      <parent link="${name}_kinect_rgb_link"/>
-      <child link="${name}_kinect_rgb_optical_frame"/>
-    </joint>
-    <link name="${name}_kinect_rgb_optical_frame"/>
-    <!-- gazebo extensions -->
-    <xacro:kinect_rgb_gazebo_v0 link_name="${name}_kinect_rgb_link" frame_name="${name}_kinect_rgb_optical_frame" camera_name="head_mount_kinect" />
   </xacro:macro>
 </root>

Commit message: recalibrate trixi + add head_mount_kinect2_joint to calibration yaml

File: tams_pr2_description/robots/trixi.urdf.xacro (robot description, xacro)
@@ -132,5 +132,11 @@
   </xacro:wge100_camera_v0>
   <xacro:kinect2_v0 name="head_mount" parent="head_plate_frame" >
-    <origin xyz="-0.137376 0 0.091746" rpy="0 0 0" />
+    <xacro:unless value="${'head_mount_kinect2_joint_x' in calib.keys()}">
+      <origin xyz="-0.137376 0 0.091746" rpy="0 0 0" />
+    </xacro:unless>
+    <xacro:if value="${'head_mount_kinect2_joint_x' in calib.keys()}">
+      <origin xyz="${calib['head_mount_kinect2_joint_x']} ${calib['head_mount_kinect2_joint_y']} ${calib['head_mount_kinect2_joint_z']}"
+              rpy="${calib['head_mount_kinect2_joint_a']} ${calib['head_mount_kinect2_joint_b']} ${calib['head_mount_kinect2_joint_c']}" />
+    </xacro:if>
   </xacro:kinect2_v0>
 </robot>

Commit message: fix deprecation warning Using load_yaml() directly is deprecated. Use xacro.load_yaml() instead.

File: tams_pr2_description/robots/trixi.urdf.xacro (robot description, xacro)
@@ -37,5 +37,5 @@
   <xacro:include filename="$(find tams_motorhand_description)/urdf/tams_motorhand.urdf.xacro" />
   <xacro:arg name="calib_config" default="$(find tams_pr2_description)/config/calibration_config.yaml" />
-  <xacro:property name="calib" value="${load_yaml('$(arg calib_config)')}"/>
+  <xacro:property name="calib" value="${xacro.load_yaml('$(arg calib_config)')}"/>
   <!-- TAMS' Shadow additions -->
   <xacro:include filename="$(find sr_description)/hand/xacro/full_hand.urdf.xacro" />

Commit message: remove xtion camera
we unmounted the camera and it was never used :/

File: tams_pr2_description/robots/trixi.urdf.xacro (robot description, xacro)
@@ -32,5 +32,4 @@
   <xacro:include filename="$(find tams_pr2_description)/urdf/ft_forearm/pr2_ft_forearm.urdf.xacro" />
   <xacro:include filename="$(find tams_pr2_description)/urdf/tams_pr2_shadow_adapter.urdf.xacro" />
-  <xacro:include filename="$(find tams_pr2_description)/urdf/xtion_camera.urdf.xacro" />
   <xacro:include filename="$(find pr2_description)/urdf/sensors/kinect2.urdf.xacro" />
   <xacro:include filename="$(find tams_pr2_description)/urdf/turn_gravity_off.urdf.xacro" />
@@ -62,7 +61,4 @@
     <origin xyz="0.0 0.0 0.0" rpy="0 0 0" />
   </xacro:pr2_head_sensor_package_v0>
-  <xacro:xtion_camera name="head_mount_xtion" parent="head_plate_frame">
-    <origin xyz="0.03 0.02 0.091746" rpy="0 0 0" />
-  </xacro:xtion_camera>
   <!-- Projector -->
   <xacro:projector_wg6802418_v0 name="projector_wg6802418" parent="head_plate_frame" >

Commit message: add symmetric l_eye / r_eye frames
These can be used in tams_pr2_neopixel to specify the led markers

File: tams_pr2_description/robots/trixi.urdf.xacro (robot description, xacro)
@@ -54,4 +54,16 @@
             rpy="0.0 0.0 0.0" />
   </xacro:pr2_head_v0>
+  <link name="l_eye" />
+  <link name="r_eye" />
+  <joint name="l_eye_joint" type="fixed">
+    <parent link="head_plate_frame" />
+	 <child link="l_eye" />
+	 <origin xyz="0.048 0.110 0.055" rpy="${M_PI/2} 0.0 ${M_PI/2}" />
+  </joint>
+  <joint name="r_eye_joint" type="fixed">
+    <parent link="head_plate_frame" />
+	 <child link="r_eye" />
+	 <origin xyz="0.048 -0.110 0.055" rpy="${M_PI/2} 0.0 ${M_PI/2}" />
+  </joint>
   <!-- Camera package: double stereo, prosilica -->
   <xacro:pr2_head_sensor_package_v0 name="sensor_mount" hd_frame_name="high_def"
