Commit message: remove kinect2 from description
it's not mounted anymore

File: tams_pr2_description/robots/tams_pr2.urdf.xacro (robot description, xacro)
@@ -32,5 +32,4 @@
   <xacro:include filename="$(find tams_pr2_description)/urdf/ft_forearm/pr2_ft_forearm.urdf.xacro" />
   <xacro:include filename="$(find tams_pr2_description)/urdf/tams_pr2_shadow_adapter.urdf.xacro" />
-  <xacro:include filename="$(find pr2_description)/urdf/sensors/kinect2.urdf.xacro" />
   <xacro:include filename="$(find tams_pr2_description)/urdf/turn_gravity_off.urdf.xacro" />
   <xacro:include filename="$(find tams_motorhand_description)/urdf/tams_motorhand.urdf.xacro" />
@@ -139,12 +138,3 @@
     <origin xyz=".135 0 .044" rpy="${-M_PI/2} ${-32.25*M_PI/180} 0" />
   </xacro:wge100_camera_v0>
-  <xacro:kinect2_v0 name="head_mount" parent="head_plate_frame" >
-    <xacro:unless value="${'head_mount_kinect2_joint_x' in calib.keys()}">
-      <origin xyz="-0.137376 0 0.091746" rpy="0 0 0" />
-    </xacro:unless>
-    <xacro:if value="${'head_mount_kinect2_joint_x' in calib.keys()}">
-      <origin xyz="${calib['head_mount_kinect2_joint_x']} ${calib['head_mount_kinect2_joint_y']} ${calib['head_mount_kinect2_joint_z']}"
-              rpy="${calib['head_mount_kinect2_joint_a']} ${calib['head_mount_kinect2_joint_b']} ${calib['head_mount_kinect2_joint_c']}" />
-    </xacro:if>
-  </xacro:kinect2_v0>
 </robot>

Commit message: minor cleanup in urdf

File: tams_pr2_description/robots/tams_pr2.urdf.xacro (robot description, xacro)
@@ -33,4 +33,5 @@
   <xacro:include filename="$(find tams_pr2_description)/urdf/tams_pr2_shadow_adapter.urdf.xacro" />
   <xacro:include filename="$(find tams_pr2_description)/urdf/turn_gravity_off.urdf.xacro" />
+  <xacro:include filename="$(find tams_pr2_description)/urdf/tams_eye.urdf.xacro" />
   <xacro:include filename="$(find tams_motorhand_description)/urdf/tams_motorhand.urdf.xacro" />
   <xacro:arg name="calib_config" default="$(find tams_pr2_description)/config/calibration_config.yaml" />
@@ -53,16 +54,10 @@
             rpy="0.0 0.0 0.0" />
   </xacro:pr2_head_v0>
-  <link name="l_eye" />
-  <link name="r_eye" />
-  <joint name="l_eye_joint" type="fixed">
-    <parent link="head_plate_frame" />
-	 <child link="l_eye" />
-	 <origin xyz="0.048 0.110 0.055" rpy="${M_PI/2} 0.0 ${M_PI/2}" />
-  </joint>
-  <joint name="r_eye_joint" type="fixed">
-    <parent link="head_plate_frame" />
-	 <child link="r_eye" />
-	 <origin xyz="0.048 -0.110 0.055" rpy="${M_PI/2} 0.0 ${M_PI/2}" />
-  </joint>
+  <xacro:tams_eye name="l_eye" parent="head_plate_frame">
+    <origin xyz="0.048 0.110 0.055" rpy="${M_PI/2} 0.0 ${M_PI/2}" />
+  </xacro:tams_eye>
+  <xacro:tams_eye name="r_eye" parent="head_plate_frame">
+    <origin xyz="0.048 -0.110 0.055" rpy="${M_PI/2} 0.0 ${M_PI/2}" />
+  </xacro:tams_eye>
   <!-- Camera package: double stereo, prosilica -->
   <xacro:pr2_head_sensor_package_v0 name="sensor_mount" hd_frame_name="high_def"
@@ -97,6 +92,6 @@
   <joint name="rh_adapter_hand_joint" type="fixed">
     <parent link="rh_adapter_link" />
-	 <child link="rh_forearm" />
-	 <origin xyz="0 0 0" rpy="0 ${-M_PI/2} ${M_PI}" />
+    <child link="rh_forearm" />
+    <origin xyz="0 0 0" rpy="0 ${-M_PI/2} ${M_PI}" />
   </joint>
   <!-- This is necessary to simulate the 'floating' of the right arm-->

Commit message: restructure head mounts & add new cameras

File: tams_pr2_description/robots/tams_pr2.urdf.xacro (robot description, xacro)
@@ -33,5 +33,5 @@
   <xacro:include filename="$(find tams_pr2_description)/urdf/tams_pr2_shadow_adapter.urdf.xacro" />
   <xacro:include filename="$(find tams_pr2_description)/urdf/turn_gravity_off.urdf.xacro" />
-  <xacro:include filename="$(find tams_pr2_description)/urdf/tams_eye.urdf.xacro" />
+  <xacro:include filename="$(find tams_pr2_description)/urdf/tams_head_additions.urdf.xacro" />
   <xacro:include filename="$(find tams_motorhand_description)/urdf/tams_motorhand.urdf.xacro" />
   <xacro:arg name="calib_config" default="$(find tams_pr2_description)/config/calibration_config.yaml" />
@@ -54,10 +54,4 @@
             rpy="0.0 0.0 0.0" />
   </xacro:pr2_head_v0>
-  <xacro:tams_eye name="l_eye" parent="head_plate_frame">
-    <origin xyz="0.048 0.110 0.055" rpy="${M_PI/2} 0.0 ${M_PI/2}" />
-  </xacro:tams_eye>
-  <xacro:tams_eye name="r_eye" parent="head_plate_frame">
-    <origin xyz="0.048 -0.110 0.055" rpy="${M_PI/2} 0.0 ${M_PI/2}" />
-  </xacro:tams_eye>
   <!-- Camera package: double stereo, prosilica -->
   <xacro:pr2_head_sensor_package_v0 name="sensor_mount" hd_frame_name="high_def"
@@ -67,4 +61,6 @@
     <origin xyz="0.0 0.0 0.0" rpy="0 0 0" />
   </xacro:pr2_head_sensor_package_v0>
+  <!-- TAMS's additions to the head -->
+  <xacro:tams_head_additions parent="head_plate_frame" />
   <!-- Projector -->
   <xacro:projector_wg6802418_v0 name="projector_wg6802418" parent="head_plate_frame" >
